File: Brakelight_1.1/BrakeLight.kicad_pcb (KiCad board)
At the start: 2 copper layers, 99 x 20 mm, 37 parts, among them J2 Conn_01x01_Socket, J3 Conn_01x01_Socket, U1 LM317MABDTG

Commit message: Upgrade old version
Parts:
- added G***: LOGO, Logos:SignatureBox30mm, B.Cu at (138.9, 146.8)
- moved R5 14.3 mm to (139.7, 156.1)
Routing:
- net Net-(D17-A): track 4.78 -> 19.8 mm
- net /ADJ: track 106.8 -> 106.0 mm, vias 2 -> 0
Other:
- board text added: "Brake_Light V2.0"
- board text added: "Michał Błotniak"
